File: Miniboard.kicad_pcb (KiCad board)
At the start: 2 copper layers, 51 x 21.5 mm, 77 parts, among them J1 USB_C_Receptacle_USB2.0, SW1 RESET, U1 ATmega16U4-A, Y1 16MHz

Commit message: Routed
Parts:
- removed D10, D3, D4: 1N4148, Diode_SMD:D_SOD-323_HandSoldering
- added H2: MountingHole, Miniboard:MountingHole, F.Cu at (102.5, 88.3)
- C1, C2, C3, C4, C5, C8, C9: footprint Resistor_SMD:R_0402_1005Metric -> Capacitor_SMD:C_0402_1005Metric
- C6, C7: value 20pF -> 12pF; footprint Resistor_SMD:R_0402_1005Metric -> Capacitor_SMD:C_0402_1005Metric
- moved G*** 12.3 mm to (107.1, 85.3)
- moved H1 2.06 mm to (147.8, 79.0)
- moved SW1 1.37 mm to (115.8, 83.2), turned to -90 degrees
- moved R5 1.21 mm to (102.1, 79.3), turned to -135 degrees
- moved LD1 1.15 mm to (101.1, 78.3), turned to -135 degrees
- moved D2 0.79 mm to (143.3, 81.7), turned to 135 degrees
- moved R1 0.25 mm to (115.1, 78.5)
Connections:
- KEY23 pad 2: Net-(D3-A) -> ROW_2
- KEY34 pad 2: Net-(D4-A) -> ROW_3
- KEY44 pad 2: Net-(D10-A) -> ROW_4
- U1 pad 11: unconnected-(U1-PB3-Pad11) -> LED
- U1 pad 12: unconnected-(U1-PB7-Pad12) -> ROW_2
- U1 pad 18: unconnected-(U1-PD0-Pad18) -> ROW_1
- U1 pad 20: unconnected-(U1-PD2-Pad20) -> ROW_0
- U1 pad 22: unconnected-(U1-PD5-Pad22) -> COL_0
- U1 pad 25: unconnected-(U1-PD4-Pad25) -> COL_1
- U1 pad 27: unconnected-(U1-PD7-Pad27) -> COL_2
- U1 pad 28: unconnected-(U1-PB4-Pad28) -> COL_3
- U1 pad 30: unconnected-(U1-PB6-Pad30) -> COL_4
- U1 pad 31: unconnected-(U1-PC6-Pad31) -> COL_5
- U1 pad 36: unconnected-(U1-PF7-Pad36) -> COL_7
- U1 pad 37: unconnected-(U1-PF6-Pad37) -> COL_8
- U1 pad 38: unconnected-(U1-PF5-Pad38) -> COL_9
- U1 pad 39: unconnected-(U1-PF4-Pad39) -> COL_10
- U1 pad 40: unconnected-(U1-PF1-Pad40) -> ROW_3
- U1 pad 41: unconnected-(U1-PF0-Pad41) -> ROW_4
- U1 pad 9: unconnected-(U1-PB1-Pad9) -> COL_6
Routing:
- net GND: track 10.6 -> 138.3 mm, vias 0 -> 17
- net COL_2: track 0.00 -> 86.9 mm, vias 0 -> 6
- net COL_1: track 0.00 -> 85.1 mm, vias 0 -> 1
- net COL_0: track 0.00 -> 68.7 mm, vias 0 -> 1
- net COL_3: track 0.00 -> 63.0 mm, vias 0 -> 3
- net COL_4: track 0.00 -> 49.9 mm, vias 0 -> 3
- net ROW_0: track 0.00 -> 45.6 mm, vias 0 -> 3
- net LED: track 0.00 -> 45.2 mm, vias 0 -> 2
- net +5V: track 8.91 -> 53.0 mm
- net COL_7: track 0.00 -> 39.8 mm, vias 0 -> 4
- net ROW_3: track 54.2 -> 91.7 mm, vias 0 -> 3
- net COL_5: track 0.00 -> 35.6 mm, vias 0 -> 1
- net COL_9: track 0.00 -> 26.8 mm, vias 0 -> 2
- net COL_8: track 0.00 -> 26.7 mm, vias 0 -> 3
- net COL_6: track 0.00 -> 23.6 mm, vias 0 -> 1
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- added copper zone on B.Cu, net GND
- added copper zone on F.Cu, net GND
Other:
- outline, holes or cut-outs redrawn
- board text added: "${TITLE}"
- board text added: ":"
- board text added: "<"
- board text added: ">"
- board text added: "?"
- board text added: "A"
- board text added: "Alt"
- board text added: "B"
- board text added: "C"
- board text added: "Ctrl"
- board text added: "D"
- board text added: "Del"
- board text added: "E"
- board text added: "Enter"
- board text added: "Esc"
- board text added: "G"
- board text added: "H"
- board text added: "I"
- board text added: "JLCJLCJLCJLC"
- board text added: "K"
- board text added: "L"
- board text added: "M"
- board text added: "N"
- board text added: "O"
- board text added: "P"
- board text added: "Q"
- board text added: "R"
- board text added: "S"
- board text added: "Shift"
- board text added: "Super"
- board text added: "T"
- board text added: "U"
- board text added: "V"
- board text added: "W"
- board text added: "X"
- board text added: "Y"
- board text added: "Z"
- board text added: "v${REVISION}"
- board text added: "~{F}"
- board text added: "~{J}"
