File: Miniboard.kicad_sch (KiCad schematic)
At the start: 9 parts, among them J1 USB_C_Receptacle_USB2.0

Commit message: Routed
Parts:
- added C1, C2, C9: 1uF, Capacitor_SMD:C_0402_1005Metric, symbol Device:C
- added C3, C4, C5, C8: 100nF, Capacitor_SMD:C_0402_1005Metric, symbol Device:C
- added C6, C7: 12pF, Capacitor_SMD:C_0402_1005Metric, symbol Device:C_Small
- added H2: MountingHole, Miniboard:MountingHole, symbol Mechanical:MountingHole
- added R6: 10k, Resistor_SMD:R_0402_1005Metric, symbol Device:R
- added SW1: RESET, Button_Switch_SMD:SW_SPST_B3U-1000P, symbol Switch:SW_Push
- added U2: ATmega32U4-A, Package_QFP:TQFP-44_10x10mm_P0.8mm, symbol MCU_Microchip_ATmega:ATmega32U4-A
- added Y1: 16MHz, Crystal:Crystal_SMD_3225-4Pin_3.2x2.5mm, symbol Device:Crystal_GND24_Small
Connections:
- net +5V: now also C1.1, C2.1, C3.1, C4.1, C5.1, R6.1, U2.14 (VCC), U2.2 (UVCC), U2.24 (AVCC), U2.34 (VCC), U2.44 (AVCC), U2.7 (VBUS)
- net GND: now also C1.2, C2.2, C3.2, C4.2, C5.2, C6.1, C7.1, C8.2, C9.2, SW1.1, U2.15 (GND), U2.23 (GND), U2.33 (~{HWB}/PE2), U2.35 (GND), U2.43 (GND), U2.5 (UGND), Y1.2, Y1.4
- net LED: now also U2.11 (PB3)
- net USB_D+: now also U2.4 (D+)
- net USB_D-: now also U2.3 (D-)
- new net: C7.2, U2.16 (XTAL2), Y1.1
- new net: C6.2, U2.17 (XTAL1), Y1.3
- new net: C8.1, U2.42 (AREF)
- new net: C9.1, U2.6 (UCAP)
- new net COL_0: U2.22 (PD5)
- new net COL_1: U2.25 (PD4)
- new net COL_10: U2.39 (PF4)
- new net COL_2: U2.27 (PD7)
- new net COL_3: U2.28 (PB4)
- new net COL_4: U2.30 (PB6)
- new net COL_5: U2.31 (PC6)
- new net COL_6: U2.9 (PB1)
- new net COL_7: U2.36 (PF7)
- new net COL_8: U2.37 (PF6)
- new net COL_9: U2.38 (PF5)
- new net RESET: R6.2, SW1.2, U2.13 (~{RESET})
- new net ROW_0: U2.20 (PD2)
- new net ROW_1: U2.18 (PD0)
- new net ROW_2: U2.12 (PB7)
- new net ROW_3: U2.40 (PF1)
- new net ROW_4: U2.41 (PF0)
- no-connect marks 2 -> 10
Other:
- removed sheet MCU
- note removed: "USB"
- title: Calcite52 Keyboard -> Miniboard
- moved on the sheet: F1, J1, LD1, R1, R2, R3, R4, R5
