File: key_matrix.kicad_sch (KiCad schematic)
At the start: 54 parts

Commit message: Routed
Parts:
- removed D10, D8, D9: 1N4148, Diode_SMD:D_SOD-323_HandSoldering, symbol Diode:1N4148
- KEY10, KEY11, KEY12, KEY13, KEY14, KEY15, KEY16, KEY17, KEY18, KEY19, KEY20, KEY21, KEY22, KEY23, KEY24, KEY25, KEY26, KEY27, KEY28, KEY29, KEY3, KEY30, KEY31, KEY32, KEY33, KEY34, KEY35, KEY36, KEY37, KEY38, KEY39, KEY4, KEY40, KEY41, KEY42, KEY43, KEY44, KEY5, KEY6, KEY7, KEY8, KEY9: LCSC (none) -> C256105
Connections:
- net ROW_2: now also KEY23.2; no longer D3.1 (K)
- net ROW_3: now also KEY34.2; no longer D4.1 (K)
- net ROW_4: now also D3.1 (K), D4.1 (K), KEY44.2
- net at KEY38.2: now also D6.2 (A)
- net at KEY39.2: now also D7.2 (A)
- net at D3.2 (A): now also KEY35.2; no longer KEY23.2
- net at KEY37.2: now also D5.2 (A); no longer D7.2 (A)
- net at D4.2 (A): now also KEY36.2; no longer KEY34.2
