File: rev1/Miniboard.kicad_pcb (KiCad board)
At the start: 2 copper layers, 51 x 21.5 mm, 75 parts, among them J1 USB_C_Receptacle_USB2.0, SW1 RESET, U1 ATmega16U4-A, Y1 16MHz

Commit message: Update Rev1.0 silkscreen
Parts:
- removed G***: LOGO, LOGO
- U1: value ATmega16U4-A -> ATmega32U4-A
- renumbered D5 to D3, D6 to D4, D7 to D5, D8 to D6, D9 to D7, R6 to R5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
