File: rev2/Miniboard.kicad_pcb (KiCad board)
At the start: 4 copper layers, 50 x 18 mm, 75 parts, among them J1 USB_C_Receptacle_USB2.0, SW1 RESET, U1 ATmega32U4-M, Y1 16MHz

Commit message: Update Rev2
Parts:
- moved G*** 62.3 mm to (145.3, 83.2)
Connections:
- J1 pad A1: ROW_2 -> GND
- J1 pad B12: ROW_2 -> GND
- R1 pad 2: ROW_2 -> GND
Routing:
- net GND: track 111.1 -> 117.3 mm
- net ROW_2: track 88.5 -> 83.7 mm
- net COL_2: track 50.4 -> 51.7 mm
- net ROW_4: track 65.5 -> 66.8 mm
- net COL_3: track 45.6 -> 46.7 mm
- net COL_0: track 61.5 -> 62.5 mm
- net COL_4: track 42.9 -> 43.7 mm
- net COL_8: track 24.3 -> 25.0 mm
- added copper zone on F.Cu, net GND
- removed copper zone on F.Cu, net (none)
Other:
- outline, holes or cut-outs redrawn
- board text removed: "1"
- board text removed: "2"
- board text removed: "3"
- board text removed: "F1"

Commit message: Update BOM
Parts:
- R6: value 10k -> 5.1k
