File: rev2/Miniboard.kicad_sch (KiCad schematic)
At the start: 23 parts, among them J1 USB_C_Receptacle_USB2.0, SW1 RESET, U1 ATmega32U4-M, Y1 16MHz

Commit message: Update BOM
Parts:
- C1, C2, C9: LCSC (none) -> C52923; MFR. Part # (none) -> CL05A105KA5NQNC
- C3, C4, C5, C8: LCSC (none) -> C1525; MFR. Part # (none) -> CL05B104KO5NNNC
- C6, C7: LCSC (none) -> C1547; MFR. Part # (none) -> 0402CG120J500NT
- J1: LCSC C165948 -> C709031; MFR. Part # TYPE-C-31-M-12 -> 918-418K2023S40023
- R3, R4: LCSC C25905 -> C482106; MFR. Part # 0402WGF5101TCE -> CRCW040222R0FKED
- R5: LCSC C11702 -> C25905; MFR. Part # 0402WGF1001TCE -> 0402WGF5101TCE
- R6: value 10k -> 5.1k; LCSC (none) -> C25905; MFR. Part # (none) -> 0402WGF5101TCE
- SW1: LCSC (none) -> C231329; MFR. Part # (none) -> B3U-1000P
- U1: LCSC (none) -> C112161; MFR. Part # (none) -> ATMEGA32U4-MU
- Y1: LCSC (none) -> C2965579; MFR. Part # (none) -> XL7EL89COI-111YLC-16M
Changed lines of the file:
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@@
+      (effects (font (size 1.27 1.27)) hide)
+    )
+    (property "LCSC" "C1525" (at 115.57 41.91 0)
+      (effects (font (size 1.27 1.27)) hide)
+    )
+    (property "MFR. Part #" "CL05B104KO5NNNC" (at 115.57 41.91 0)
       (effects (font (size 1.27 1.27)) hide)
     )
@@
     )
     (property "Datasheet" "~" (at 66.04 41.91 0)
+      (effects (font (size 1.27 1.27)) hide)
+    )
+    (property "LCSC" "C52923" (at 66.04 41.91 0)
+      (effects (font (size 1.27 1.27)) hide)
+    )
+    (property "MFR. Part #" "CL05A105KA5NQNC" (at 66.04 41.91 0)
       (effects (font (size 1.27 1.27)) hide)
     )
@@
     )
   )
-  (symbol (lib_id "Device:R") (at 71.12 170.18 0) (unit 1)
-    (in_bom yes) (on_board yes) (dnp no) (fields_autoplaced)
+  (symbol (lib_id "power:GND") (at 106.68 184.15 0) (unit 1)
+    (in_bom yes) (on_board yes) (dnp no)
+    (property "Reference" "#PWR04" (at 106.68 190.5 0)
+      (effects (font (size 1.27 1.27)) hide)
+    )
+    (property "Value" "GND" (at 106.68 187.96 0)
+      (effects (font (size 1.27 1.27)))
+    )
+    (property "Footprint" "" (at 106.68 184.15 0)
+      (effects (font (size 1.27 1.27)) hide)
+    )
+    (property "Datasheet" "" (at 106.68 184.15 0)
+      (effects (font (size 1.27 1.27)) hide)
+    )
+    (pin "1")
+    (instances
+      (project "Miniboard"
+        (path "/717fb49e-fed7-4c0b-8814-f6ed14872a26"
+          (reference "#PWR04") (unit 1)
+        )
+      )
+    )
+  )
+  (symbol (lib_id "Device:R") (at 71.12 170.18 0) (mirror y) (unit 1)
+    (in_bom yes) (on_board yes) (dnp no)
     (property "Reference" "R6" (at 73.66 168.91 0)
-      (effects (font (size 1.27 1.27)) (justify left))
-    )
-    (property "Value" "10k" (at 73.66 171.45 0)
-      (effects (font (size 1.27 1.27)) (justify left))
-    )
-    (property "Footprint" "Resistor_SMD:R_0402_1005Metric" (at 69.342 170.18 90)
+      (effects (font (size 1.27 1.27)) (justify right))
+    )
+    (property "Value" "5.1k" (at 73.66 171.45 0)
+      (effects (font (size 1.27 1.27)) (justify right))
+    )
+    (property "Footprint" "Resistor_SMD:R_0402_1005Metric" (at 72.898 170.18 90)
       (effects (font (size 1.27 1.27)) hide)
     )
@@
       (effects (font (size 1.27 1.27)) hide)
     )
+    (property "MFR. Part #" "0402WGF5101TCE" (at 71.12 170.18 0)
+      (effects (font (size 1.27 1.27)) hide)
+    )
+    (property "LCSC" "C25905" (at 71.12 170.18 0)
+      (effects (font (size 1.27 1.27)) hide)
+    )
     (pin "1")
     (pin "2")
@@
     )
   )
-  (symbol (lib_id "power:GND") (at 106.68 184.15 0) (unit 1)
-    (in_bom yes) (on_board yes) (dnp no)
-    (property "Reference" "#PWR04" (at 106.68 190.5 0)
-      (effects (font (size 1.27 1.27)) hide)
-    )
-    (property "Value" "GND" (at 106.68 187.96 0)
-      (effects (font (size 1.27 1.27)))
-    )
-    (property "Footprint" "" (at 106.68 184.15 0)
-      (effects (font (size 1.27 1.27)) hide)
-    )
-    (property "Datasheet" "" (at 106.68 184.15 0)
-      (effects (font (size 1.27 1.27)) hide)
-    )
-    (pin "1")
-    (instances
-      (project "Miniboard"
-        (path "/717fb49e-fed7-4c0b-8814-f6ed14872a26"
-          (reference "#PWR04") (unit 1)
-        )
-      )
-    )
-  )
   (symbol (lib_id "power:+5V") (at 71.12 166.37 0) (unit 1)
     (in_bom yes) (on_board yes) (dnp no)
@@
     )
     (property "Datasheet" "~" (at 39.37 66.04 0)
+      (effects (font (size 1.27 1.27)) hide)
+    )
+    (property "LCSC" "C1547" (at 39.37 66.04 0)
+      (effects (font (size 1.27 1.27)) hide)
+    )
+    (property "MFR. Part #" "0402CG120J500NT" (at 39.37 66.04 0)
       (effects (font (size 1.27 1.27)) hide)
     )
@@
       (effects (font (size 1.27 1.27)) hide)
     )
+    (property "LCSC" "C1547" (at 39.37 60.96 0)
+      (effects (font (size 1.27 1.27)) hide)
+    )
+    (property "MFR. Part #" "0402CG120J500NT" (at 39.37 60.96 0)
+      (effects (font (size 1.27 1.27)) hide)
+    )
     (pin "1")
     (pin "2")
@@
       (effects (font (size 1.27 1.27)) hide)
     )
-    (property "JLCPCB Part #" "" (at 228.6 57.15 0)
-      (effects (font (size 1.27 1.27)) hide)
-    )
-    (property "MFR. Part #" "0402WGF5101TCE" (at 228.6 57.15 0)
-      (effects (font (size 1.27 1.27)) hide)
-    )
-    (property "LCSC" "C25905" (at 228.6 57.15 0)
+    (property "MFR. Part #" "CRCW040222R0FKED" (at 228.6 57.15 0)
+      (effects (font (size 1.27 1.27)) hide)
+    )
+    (property "LCSC" "C482106" (at 228.6 57.15 0)
       (effects (font (size 1.27 1.27)) hide)
     )
@@
       (effects (font (size 1.27 1.27)) hide)
     )
-    (property "JLCPCB Part #" "" (at 228.6 52.07 0)
-      (effects (font (size 1.27 1.27)) hide)
-    )
-    (property "MFR. Part #" "0402WGF5101TCE" (at 228.6 52.07 0)
-      (effects (font (size 1.27 1.27)) hide)
-    )
-    (property "LCSC" "C25905" (at 228.6 52.07 0)
+    (property "MFR. Part #" "CRCW040222R0FKED" (at 228.6 52.07 0)
+      (effects (font (size 1.27 1.27)) hide)
+    )
+    (property "LCSC" "C482106" (at 228.6 52.07 0)
       (effects (font (size 1.27 1.27)) hide)
     )
@@
       (effects (font (size 1.27 1.27)) hide)
     )
+    (property "LCSC" "C231329" (at 71.12 179.07 0)
+      (effects (font (size 1.27 1.27)) hide)
+    )
+    (property "MFR. Part #" "B3U-1000P" (at 71.12 179.07 0)
+      (effects (font (size 1.27 1.27)) hide)
+    )
     (pin "1")
     (pin "2")
@@
       (effects (font (size 1.27 1.27)) hide)
     )
-    (property "JLCPCB Part #" "" (at 222.25 45.72 0)
-      (effects (font (size 1.27 1.27)) hide)
-    )
     (property "MFR. Part #" "0402WGF5101TCE" (at 222.25 45.72 0)
       (effects (font (size 1.27 1.27)) hide)
@@
       (effects (font (size 1.27 1.27)) hide)
     )
+    (property "LCSC" "C1525" (at 101.6 41.91 0)
+      (effects (font (size 1.27 1.27)) hide)
+    )
+    (property "MFR. Part #" "CL05B104KO5NNNC" (at 101.6 41.91 0)
+      (effects (font (size 1.27 1.27)) hide)
+    )
     (pin "1")
     (pin "2")
@@
     )
     (property "Datasheet" "~" (at 128.27 41.91 0)
+      (effects (font (size 1.27 1.27)) hide)
+    )
+    (property "LCSC" "C1525" (at 128.27 41.91 0)
+      (effects (font (size 1.27 1.27)) hide)
+    )
+    (property "MFR. Part #" "CL05B104KO5NNNC" (at 128.27 41.91 0)
       (effects (font (size 1.27 1.27)) hide)
     )
@@
       (effects (font (size 1.27 1.27)) hide)
     )
-    (property "MFR. Part #" "TYPE-C-31-M-12" (at 199.39 53.34 0)
-      (effects (font (size 1.27 1.27)) hide)
-    )
-    (property "LCSC" "C165948" (at 199.39 53.34 0)
+    (property "MFR. Part #" "918-418K2023S40023" (at 199.39 53.34 0)
+      (effects (font (size 1.27 1.27)) hide)
+    )
+    (property "LCSC" "C709031" (at 199.39 53.34 0)
       (effects (font (size 1.27 1.27)) hide)
     )
@@
     )
     (property "Datasheet" "http://ww1.microchip.com/downloads/en/DeviceDoc/Atmel-7766-8-bit-AVR-ATmega16U4-32U4_Datasheet.pdf" (at 82.55 93.98 0)
+      (effects (font (size 1.27 1.27)) hide)
+    )
+    (property "LCSC" "C112161" (at 82.55 93.98 0)
+      (effects (font (size 1.27 1.27)) hide)
+    )
+    (property "MFR. Part #" "ATMEGA32U4-MU" (at 82.55 93.98 0)
       (effects (font (size 1.27 1.27)) hide)
     )
@@
       (effects (font (size 1.27 1.27)) hide)
     )
+    (property "LCSC" "C2965579" (at 46.99 63.5 0)
+      (effects (font (size 1.27 1.27)) hide)
+    )
+    (property "MFR. Part #" "XL7EL89COI-111YLC-16M" (at 46.99 63.5 0)
+      (effects (font (size 1.27 1.27)) hide)
+    )
     (pin "1")
     (pin "2")
@@
     )
     (property "MFR. Part #" "SMD0805B050TF" (at 228.6 38.1 90)
-      (effects (font (size 1.27 1.27)) hide)
-    )
-    (property "JLCPCB Part #" "" (at 228.6 38.1 90)
       (effects (font (size 1.27 1.27)) hide)
     )
@@
       (effects (font (size 1.27 1.27)) hide)
     )
-    (property "MFR. Part #" "0402WGF1001TCE " (at 106.68 180.34 0)
-      (effects (font (size 1.27 1.27)) hide)
-    )
-    (property "JLCPCB Part #" "" (at 106.68 180.34 0)
-      (effects (font (size 1.27 1.27)) hide)
-    )
-    (property "LCSC" "C11702" (at 106.68 180.34 0)
+    (property "MFR. Part #" "0402WGF5101TCE" (at 106.68 180.34 0)
+      (effects (font (size 1.27 1.27)) hide)
+    )
+    (property "LCSC" "C25905" (at 106.68 180.34 0)
       (effects (font (size 1.27 1.27)) hide)
     )
@@
       (effects (font (size 1.27 1.27)) hide)
     )
+    (property "LCSC" "C52923" (at 59.69 92.71 0)
+      (effects (font (size 1.27 1.27)) hide)
+    )
+    (property "MFR. Part #" "CL05A105KA5NQNC" (at 59.69 92.71 0)
+      (effects (font (size 1.27 1.27)) hide)
+    )
     (pin "1")
     (pin "2")
@@
       (effects (font (size 1.27 1.27)) hide)
     )
+    (property "LCSC" "C1525" (at 48.26 92.71 0)
+      (effects (font (size 1.27 1.27)) hide)
+    )
+    (property "MFR. Part #" "CL05B104KO5NNNC" (at 48.26 92.71 0)
+      (effects (font (size 1.27 1.27)) hide)
+    )
     (pin "1")
     (pin "2")
@@
       (effects (font (size 1.27 1.27)) hide)
     )
-    (property "JLCPCB Part #" "" (at 222.25 43.18 0)
-      (effects (font (size 1.27 1.27)) hide)
-    )
     (property "MFR. Part #" "0402WGF5101TCE" (at 222.25 43.18 0)
       (effects (font (size 1.27 1.27)) hide)
@@
       (effects (font (size 1.27 1.27)) hide)
     )
+    (property "LCSC" "C52923" (at 54.61 41.91 0)
+      (effects (font (size 1.27 1.27)) hide)
+    )
+    (property "MFR. Part #" "CL05A105KA5NQNC" (at 54.61 41.91 0)
+      (effects (font (size 1.27 1.27)) hide)
+    )
