File: rev2/key_matrix.kicad_sch (KiCad schematic)
At the start: 51 parts

Commit message: Update BOM
Parts:
- D1, D2, D3, D4, D5, D6, D7: LCSC C81598 -> C2128; MFR. Part # 1N4148W -> 1N4148WS
- KEY1, KEY2: LCSC (none) -> C393942; MFR. Part # (none) -> TS24CA
- KEY10, KEY11, KEY12, KEY13, KEY14, KEY15, KEY16, KEY17, KEY18, KEY19, KEY20, KEY21, KEY22, KEY23, KEY24, KEY25, KEY26, KEY27, KEY28, KEY29, KEY3, KEY30, KEY31, KEY32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: MFR. Part # (none) -> 1TS015A-1800-0600-CT
